File: pcb/barkbit/barkbit.kicad_pcb (KiCad board)
At the start: 2 copper layers, 19 parts, among them J1 BATT, J2 PRG, U1 MX25R6435FM2IH0, U2 MDBT42Q, U3 TLV61225, U4 MMA8451Q

Commit message: Final board. Cleanups.
Parts:
- removed C4: 0.1uf, Capacitor_SMD:C_0805_2012Metric_Pad1.15x1.40mm_HandSolder
- added C9: 10uF, Capacitor_SMD:C_0805_2012Metric_Pad1.15x1.40mm_HandSolder, F.Cu at (151.2, 68.8)
- J1: footprint Connector_PinHeader_2.54mm:PinHeader_1x02_P2.54mm_Vertical -> barkbit:Wire_1x02_P1.27mm
- J2: footprint Connector_PinHeader_2.54mm:PinHeader_1x04_P2.54mm_Vertical -> barkbit:Wire_1x04_P1.27mm
- moved J1 50.3 mm to (161.6, 75.8), turned to 270 degrees
- moved J2 43.7 mm to (160.3, 78.1), turned to 90 degrees
- moved C6 34.5 mm to (155.2, 65.8), turned to 90 degrees
- moved C7 32.3 mm to (153.2, 72.7), turned to 90 degrees
- moved R2 31.1 mm to (152.2, 65.9), turned to 180 degrees
- moved C5 28.1 mm to (162.5, 67.1), turned to 90 degrees
- moved U1 27.2 mm to (158.9, 71.9)
- moved U4 26.8 mm to (158.0, 67.0)
- moved L1 24.8 mm to (151.1, 55.0), turned to 90 degrees
- moved R1 24.7 mm to (153.2, 68.8), turned to 270 degrees
- moved C3 24.2 mm to (151.3, 72.7), turned to 90 degrees
- moved L3 19.8 mm to (151.1, 58.8), turned to 90 degrees
- moved L2 18.9 mm to (151.3, 76.7), turned to 270 degrees
- moved C1 15.2 mm to (151.1, 62.6), turned to 270 degrees
- moved C8 13.2 mm to (158.6, 76.7), turned to 90 degrees
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Connections:
- U2 pad 13: Net-(U2-Pad13) -> /I2C_SDA
- U2 pad 14: Net-(U2-Pad14) -> /I2C_SCL
- U2 pad 15: Net-(U2-Pad15) -> /MMA_INT1
- U2 pad 16: Net-(U2-Pad16) -> /MMA_INT2
- U2 pad 20: Net-(U2-Pad20) -> /FLASH_CS
- U2 pad 21: /FLASH_CS -> /SPI_MISO
- U2 pad 22: Net-(U2-Pad22) -> /SPI_MOSI
- U2 pad 23: Net-(U2-Pad23) -> /SPI_SCK
- U2 pad 26: /SPI_SCK -> Net-(U2-Pad26)
- U2 pad 27: /SPI_MOSI -> Net-(U2-Pad27)
- U2 pad 28: /SPI_MISO -> Net-(U2-Pad28)
- U2 pad 32: /MMA_INT2 -> Net-(U2-Pad32)
- U2 pad 33: /MMA_INT1 -> Net-(U2-Pad33)
- U2 pad 34: /I2C_SDA -> Net-(U2-Pad34)
- U2 pad 35: /I2C_SCL -> Net-(U2-Pad35)
- U2 pad 36: Net-(J2-Pad4) -> Net-(J2-Pad3)
- U2 pad 37: Net-(J2-Pad3) -> Net-(J2-Pad4)
Routing:
- net +3V3: track 0.00 -> 54.1 mm, vias 0 -> 2
- net Net-(J2-Pad4): track 0.00 -> 27.1 mm
- net Net-(J2-Pad3): track 0.00 -> 26.8 mm
- net GND: track 0.00 -> 24.6 mm, vias 0 -> 13
- net /I2C_SDA: track 0.00 -> 12.8 mm
- net /SPI_MOSI: track 0.00 -> 12.7 mm
- net /SPI_MISO: track 0.00 -> 12.5 mm
- net Net-(C1-Pad1): track 0.00 -> 12.2 mm, vias 0 -> 2
- net /FLASH_CS: track 0.00 -> 11.8 mm
- net +3V0: track 0.00 -> 11.8 mm
- net /SPI_SCK: track 0.00 -> 11.3 mm
- net /I2C_SCL: track 0.00 -> 10.0 mm
- net /MMA_INT2: track 0.00 -> 8.84 mm
- net /MMA_INT1: track 0.00 -> 8.09 mm
- net Net-(L3-Pad1): track 0.00 -> 2.47 mm
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- added copper zone on B.Cu, net GND
Other:
- board outline added: 15 x 29 mm
- net class Default: clearance 0.2 -> 0.1524; trace_width 0.25 -> 0.1524; via_dia 0.8 -> 0.6858; via_drill 0.4 -> 0.3302
- rule pad_to_mask_clearance: 0.05 -> 0.0508
- rule trace_clearance: 0.2 -> 0.1524
- rule trace_min: 0.2 -> 0.1524
- rule via_min_drill: 0.3 -> 0.254
- rule via_min_size: 0.4 -> 0.508
- board text added: "FitBark 1.0"

Commit message: Cleanups.
Connections:
- net Net-(J2-Pad3) renamed /SWDCLK
- net Net-(J2-Pad4) renamed /SWDIO
